File: electronics/Mainboard.brd (EAGLE design)
At the start: 310 x 150 mm, 225 parts, among them J1 JST_PH_B3B-PH-K-S(LF)(SN), J10 JST_PH_B3B-PH-K-S(LF)(SN), J11 JST_PH_B3B-PH-K-S(LF)(SN), J12 JST_PH_B3B-PH-K-S(LF)(SN), J13 JST_PH_B3B-PH-K-S(LF)(SN), J14 JST_PH_B3B-PH-K-S(LF)(SN), J15 JST_PH_B3B-PH-K-S(LF)(SN), J16 JST_PH_B3B-PH-K-S(LF)(SN), J17 JST_PH_B3B-PH-K-S(LF)(SN), J18 JST_PH_B3B-PH-K-S(LF)(SN), J19 JST_PH_B3B-PH-K-S(LF)(SN), J2 JST_PH_B3B-PH-K-S(LF)(SN), J20 JST_PH_B3B-PH-K-S(LF)(SN), J21 JST_PH_B3B-PH-K-S(LF)(SN), J22 JST_PH_B3B-PH-K-S(LF)(SN), J23 JST_PH_B3B-PH-K-S(LF)(SN), J24 JST_PH_B3B-PH-K-S(LF)(SN), J25 JST_PH_B3B-PH-K-S(LF)(SN), J26 JST_PH_B3B-PH-K-S(LF)(SN), J27 JST_PH_B3B-PH-K-S(LF)(SN), J28 JST_PH_B3B-PH-K-S(LF)(SN), J29 JST_PH_B3B-PH-K-S(LF)(SN), J3 JST_PH_B3B-PH-K-S(LF)(SN), J30 JST_PH_B3B-PH-K-S(LF)(SN), J31 JST_PH_B3B-PH-K-S(LF)(SN), J32 JST_PH_B3B-PH-K-S(LF)(SN), J4 JST_PH_B3B-PH-K-S(LF)(SN), J5 JST_PH_B3B-PH-K-S(LF)(SN), J6 JST_PH_B3B-PH-K-S(LF)(SN), J7 JST_PH_B3B-PH-K-S(LF)(SN), J8 JST_PH_B3B-PH-K-S(LF)(SN), J9 JST_PH_B3B-PH-K-S(LF)(SN), U15 AD5360BSTZ, U16 ADR425ARZ, U18 AD7730BRUZ, U19 AD5360BSTZ, U20 ADR425ARZ, U21 AD7730BRUZ, U22 STM32F103RCT6, U23 AD7730BRUZ, U24 AD7730BRUZ, U25 AD7730BRUZ, U26 AD7730BRUZ, U27 AD7730BRUZ, U28 AD7730BRUZ, U38 AD7730BRUZ, U39 AD7730BRUZ, U4 ADR421ARZ, U40 STM32F103RCT6, U41 AD7730BRUZ, U42 AD7730BRUZ, U43 AD7730BRUZ, U44 AD7730BRUZ, U45 AD7730BRUZ, U46 AD7730BRUZ, U5 AD7616BSTZ, U6 74AHC1G04GW/T1, U7 ADR421ARZ, U8 AD7616BSTZ, U9 74AHC1G04GW/T1, X1 22-23-2031, Y3 KC2520B-C1, Y4 ABM3B, Y7 KC2520B-C1, Y8 ABM3B

Commit message: first changes to the load cell section on the board
Parts:
- moved C17 47.5 mm to (214.6, 125.4), flipped to the bottom, turned to 0 degrees
- moved C12 46.0 mm to (215.3, 121.9), flipped to the top, turned to 0 degrees
- moved U28 42.7 mm to (265.9, 99.5), flipped to the top
- moved C16 41.0 mm to (221.2, 133.1), flipped to the top
- moved Y4 36.9 mm to (217.9, 127.7), flipped to the bottom, turned to 270 degrees
- moved C11 29.9 mm to (174.1, 101.5), turned to 90 degrees
- moved C15 29.5 mm to (222.2, 114.9), turned to 270 degrees
- moved C18 28.0 mm to (223.8, 125.9), flipped to the bottom, turned to 180 degrees
- moved U22 27.3 mm to (224.9, 124.2), flipped to the top
- moved U25 26.8 mm to (230.8, 99.5), flipped to the top
- moved U18 25.8 mm to (183.9, 99.5)
- moved Y3 25.8 mm to (176.2, 102.4)
- moved U21 25.3 mm to (195.7, 99.5)
- moved U23 24.9 mm to (207.3, 99.5)
- moved U24 24.5 mm to (219.1, 99.5)
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Connections:
- net N$50 renamed LC_1_OSC_IN
- net N$51 renamed LC_1_OSC_OUT
- net BT_5_AIN1_+: now also J57.3; no longer J64.3
- net BT_5_AIN1_-: now also J57.4; no longer J64.4
- net BT_5_AIN2_+: now also J58.3; no longer J63.3
- net BT_5_AIN2_-: now also J58.4; no longer J63.4
- net BT_6_AIN1_+: now also J59.3; no longer J62.3
- net BT_6_AIN1_-: now also J59.4; no longer J62.4
- net BT_6_AIN2_+: now also J60.3; no longer J61.3
- net BT_6_AIN2_-: now also J60.4; no longer J61.4
- net BT_7_AIN1_+: now also J61.3; no longer J60.3
- net BT_7_AIN1_-: now also J61.4; no longer J60.4
- net BT_7_AIN2_+: now also J62.3; no longer J59.3
- net BT_7_AIN2_-: now also J62.4; no longer J59.4
- net BT_8_AIN1_+: now also J63.3; no longer J58.3
- net BT_8_AIN1_-: now also J63.4; no longer J58.4
- net BT_8_AIN2_+: now also J64.3; no longer J57.3
- net BT_8_AIN2_-: now also J64.4; no longer J57.4
Routing:
- net LC_1_RDY8: track 76.7 -> 12.9 mm, vias 2 -> 1
- net LC_1_SS8: track 80.0 -> 17.4 mm, vias 2 -> 1
- net LC_1_SS7: track 71.4 -> 15.7 mm, vias 2 -> 1
- net +5V: track 1444.9 -> 1395.1 mm, vias 15 -> 14
- net LC_1_RDY2: track 48.3 -> 90.6 mm, vias 3 -> 1
- net LC_1_RDY3: track 36.6 -> 77.8 mm, vias 3 -> 1
- net LC_1_RDY7: track 65.1 -> 24.6 mm, vias 2 -> 1
- net LC_1_RDY1: track 62.2 -> 102.5 mm, vias 3 -> 1
- net BT_4_AIN2_-: track 47.0 -> 6.77 mm
- net LC_1_RDY4: track 28.4 -> 66.6 mm, vias 3 -> 1
- net LC_1_SS6: track 52.9 -> 15.8 mm, vias 2 -> 1
- net MOSI: track 710.0 -> 675.7 mm
- net BT_2_AIN1_+: track 46.9 -> 12.8 mm
- net BT_4_AIN2_+: track 45.3 -> 12.6 mm
- net BT_4_AIN1_+: track 45.2 -> 12.8 mm
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
Commit message: reworked second load cell section
Parts:
- moved C59 88.4 mm to (340.0, 51.8), flipped to the bottom
- moved Y8 82.6 mm to (337.4, 53.3), flipped to the bottom
- moved C58 80.6 mm to (342.6, 51.8), flipped to the bottom
- moved C56 73.5 mm to (319.9, 53.0)
- moved C54 73.4 mm to (323.1, 53.0)
- moved C55 72.7 mm to (325.3, 53.0)
- moved SV21 67.9 mm to (192.4, 51.4)
- moved C53 58.6 mm to (319.8, 45.0), flipped to the top
- moved C57 57.9 mm to (319.8, 48.8), flipped to the top
- moved U46 42.6 mm to (265.9, 22.8), flipped to the top
- moved C52 29.0 mm to (174.1, 24.9), turned to 90 degrees
- moved U40 27.6 mm to (224.9, 50.0), flipped to the top
- moved U43 26.5 mm to (230.8, 22.8), flipped to the top
- moved U38 24.8 mm to (183.9, 22.8)
- moved Y7 24.8 mm to (176.2, 25.7)
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Connections:
- net N$109 renamed LC2_OSC_IN
- net N$110 renamed LC2_OSC_OUT
- net BT2_5_AIN1_+: now also J41.3; no longer J48.3
- net BT2_5_AIN1_-: now also J41.4; no longer J48.4
- net BT2_5_AIN2_+: now also J42.3; no longer J47.3
- net BT2_5_AIN2_-: now also J42.4; no longer J47.4
- net BT2_6_AIN1_+: now also J43.3; no longer J46.3
- net BT2_6_AIN1_-: now also J43.4; no longer J46.4
- net BT2_6_AIN2_+: now also J44.3; no longer J45.3
- net BT2_6_AIN2_-: now also J44.4; no longer J45.4
- net BT2_7_AIN1_+: now also J45.3; no longer J44.3
- net BT2_7_AIN1_-: now also J45.4; no longer J44.4
- net BT2_7_AIN2_+: now also J46.3; no longer J43.3
- net BT2_7_AIN2_-: now also J46.4; no longer J43.4
- net BT2_8_AIN1_+: now also J47.3; no longer J42.3
- net BT2_8_AIN1_-: now also J47.4; no longer J42.4
- net BT2_8_AIN2_+: now also J48.3; no longer J41.3
- net BT2_8_AIN2_-: now also J48.4; no longer J41.4
Routing:
- net +5V: track 1395.1 -> 1307.3 mm, vias 14 -> 11
- net LC_2_SS8: track 80.0 -> 10.6 mm, vias 2 -> 0
- net LC_2_RDY8: track 76.6 -> 8.04 mm, vias 2 -> 1
- net DVCC: track 1377.2 -> 1312.7 mm, vias 19 -> 16
- net LC_2_SS7: track 71.4 -> 13.2 mm, vias 2 -> 1
- net LC_2_RDY7: track 64.6 -> 20.0 mm, vias 2 -> 1
- net LC_2_SS6: track 52.9 -> 13.2 mm, vias 2 -> 1
- net LC_2_SS1: track 50.2 -> 12.5 mm
- net LC_2_RDY2: track 48.3 -> 79.9 mm, vias 3 -> 1
- net LC_2_RDY3: track 36.6 -> 67.9 mm, vias 3 -> 1
- net BT2_4_AIN2_-: track 36.8 -> 6.77 mm
- net LC_2_RDY1: track 62.2 -> 91.8 mm, vias 3 -> 1
- net LC_2_SPI1_MOSI: track 125.4 -> 95.8 mm, vias 11 -> 8
- net LC_2_RDY4: track 28.4 -> 55.9 mm, vias 3 -> 1
- net LC_2_SS5: track 40.1 -> 13.2 mm, vias 2 -> 1
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Other:
- board text added: "Hitzmann 2018 rev. 2.0"
- board text removed: "Hitzmann 2018 rev. 1.1"

Commit message: load cell sections done
Parts:
- moved C58 128.0 mm to (214.6, 48.7), turned to 0 degrees
- moved Y8 119.4 mm to (217.9, 51.0), turned to 270 degrees
- moved C59 116.3 mm to (223.8, 49.2), turned to 180 degrees
- moved C57 104.5 mm to (215.3, 45.5), turned to 180 degrees
- moved C56 98.8 mm to (221.2, 56.4)
- moved C53 97.8 mm to (222.2, 38.2)
- moved C55 91.5 mm to (233.8, 52.9), turned to 45 degrees
- moved C54 90.0 mm to (233.8, 40.8), turned to 315 degrees
- moved SV21 50.8 mm to (243.1, 55.1), turned to 270 degrees
- moved LED1 11.0 mm to (274.3, 121.5)
- moved LED2 11.0 mm to (280.1, 121.5)
- moved LED3 11.0 mm to (286.0, 121.5)
- moved LED4 11.0 mm to (291.9, 121.5)
- moved R1 7.80 mm to (286.0, 96.8)
- moved R10 7.80 mm to (291.9, 96.8)
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Connections:
- net LC2_OSC_IN renamed LC_2_OSC_IN
- net LC2_OSC_OUT renamed LC_2_OSC_OUT
- removed net LC_1_RDY8: U22.14, U28.20
- removed net LC_1_SS1: U18.19, U22.40
- removed net LC_1_SS2: U21.19, U22.39
- removed net LC_1_SS3: U22.38, U23.19
- removed net LC_1_SS4: U22.37, U24.19
- removed net LC_1_SS5: U22.11, U25.19
- removed net LC_1_SS6: U22.10, U26.19
- removed net LC_1_SS7: U22.9, U27.19
- removed net LC_1_SS8: U22.8, U28.19
- removed net LC_2_RDY8: U40.14, U46.20
- removed net LC_2_SS1: U38.19, U40.40
- removed net LC_2_SS2: U39.19, U40.39
- removed net LC_2_SS3: U40.38, U41.19
- removed net LC_2_SS4: U40.37, U42.19
- removed net LC_2_SS5: U40.11, U43.19
- removed net LC_2_SS6: U40.10, U44.19
- removed net LC_2_SS7: U40.9, U45.19
- removed net LC_2_SS8: U40.8, U46.19
- removed net PB7: U22.59, U40.59
- new net LC_1_CS0: U18.19, U22.14
- new net LC_1_CS1: U21.19, U22.15
- new net LC_1_CS2: U22.16, U23.19
- new net LC_1_CS3: U22.24, U24.19
- new net LC_1_CS4: U22.25, U25.19
- new net LC_1_CS5: U22.26, U26.19
- new net LC_1_CS6: U22.27, U27.19
- new net LC_1_CS7: U22.28, U28.19
- new net LC_1_PB7: U22.59
- new net LC_1_RDY0: U18.20, U22.45
- new net LC_2_CS0: U38.19, U40.14
- new net LC_2_CS1: U39.19, U40.15
- new net LC_2_CS2: U40.16, U41.19
- new net LC_2_CS3: U40.24, U42.19
- new net LC_2_CS4: U40.25, U43.19
- new net LC_2_CS5: U40.26, U44.19
- new net LC_2_CS6: U40.27, U45.19
- new net LC_2_CS7: U40.28, U46.19
- new net LC_2_PB7: U40.59
- new net LC_2_RDY0: U38.20, U40.45
- net LC_1_RDY1: now also U21.20; no longer U18.20
- net LC_1_RDY2: now also U23.20; no longer U21.20
- net LC_1_RDY3: now also U24.20; no longer U23.20
- net LC_1_RDY4: now also U22.41, U25.20; no longer U22.45, U24.20
- net LC_1_RDY5: now also U22.40, U26.20; no longer U22.17, U25.20
- net LC_1_RDY6: now also U22.39, U27.20; no longer U22.16, U26.20
- net LC_1_RDY7: now also U22.38, U28.20; no longer U22.15, U27.20
- net LC_2_RDY1: now also U39.20; no longer U38.20
- net LC_2_RDY2: now also U41.20; no longer U39.20
- net LC_2_RDY3: now also U42.20; no longer U41.20
- net LC_2_RDY4: now also U40.41, U43.20; no longer U40.45, U42.20
- net LC_2_RDY5: now also U40.40, U44.20; no longer U40.17, U43.20
- net LC_2_RDY6: now also U40.39, U45.20; no longer U40.16, U44.20
- net LC_2_RDY7: now also U40.38, U46.20; no longer U40.15, U45.20
Routing:
- net DVCC: track 1312.7 -> 1493.6 mm, vias 16 -> 17
- net LC_1_RDY0: track 0.00 -> 164.9 mm, vias 0 -> 2
- net LC_2_RDY0: track 0.00 -> 164.9 mm, vias 0 -> 2
- net +5V: track 1307.3 -> 1380.2 mm, vias 11 -> 13
- net LC_2_CS7: track 0.00 -> 62.6 mm
- net LC_1_CS7: track 0.00 -> 62.6 mm
- net LC_2_RDY1: track 91.8 -> 150.8 mm, vias 1 -> 2
- net LC_2_RDY2: track 79.9 -> 136.7 mm, vias 1 -> 2
- net LC_2_CS6: track 0.00 -> 55.6 mm, vias 0 -> 2
- net LC_1_CS6: track 0.00 -> 55.6 mm, vias 0 -> 2
- net LC_2_RDY3: track 67.9 -> 122.6 mm, vias 1 -> 2
- net LC_2_RDY4: track 55.9 -> 108.4 mm, vias 1 -> 2
- net LC_2_RDY5: track 44.0 -> 94.3 mm, vias 1 -> 2
- net LC_1_RDY1: track 102.5 -> 150.8 mm, vias 1 -> 2
- net LC_1_CS0: track 0.00 -> 48.2 mm, vias 0 -> 2
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
Commit message: reworked first dac
Parts:
- moved C21 34.8 mm to (146.9, 117.0), turned to 90 degrees
- moved C22 32.2 mm to (153.4, 112.5)
- moved C137 32.0 mm to (152.8, 110.5)
- moved C136 30.9 mm to (144.9, 116.3), turned to 90 degrees
- moved U19 22.9 mm to (140.4, 106.0), turned to 315 degrees
- moved C143 20.2 mm to (143.7, 95.5), flipped to the bottom
- moved C147 19.8 mm to (144.3, 100.8), flipped to the bottom
- moved C24 18.0 mm to (146.2, 94.9), flipped to the bottom, turned to 270 degrees
- moved C141 17.7 mm to (126.1, 113.1)
- moved C145 17.6 mm to (126.1, 108.5)
- moved C151 17.1 mm to (126.1, 102.7), turned to 270 degrees
- moved C26 16.9 mm to (122.8, 107.9)
- moved C23 16.7 mm to (122.8, 113.8)
- moved C25 16.6 mm to (146.9, 101.4), flipped to the bottom, turned to 270 degrees
- moved C10 14.3 mm to (122.8, 102.0), turned to 270 degrees
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Routing:
- net SS_DAC_2: track 84.0 -> 121.6 mm
- net MISO: track 649.0 -> 684.9 mm
- net SCLK: track 633.9 -> 669.5 mm
- net MOSI: track 655.8 -> 691.3 mm
- net DVCC: track 1493.6 -> 1526.3 mm
- net DAC2_5: track 53.8 -> 22.4 mm
- net DAC2_6: track 56.7 -> 26.3 mm
- net DAC2_7: track 59.6 -> 29.7 mm
- net DAC2_4: track 48.1 -> 18.9 mm
- net DAC2_3: track 45.9 -> 17.3 mm
- net DAC2_2: track 44.1 -> 16.1 mm
- net DAC2_1: track 42.3 -> 16.9 mm
- net DAC2_0: track 40.4 -> 16.8 mm
- net LDAC: track 212.4 -> 234.3 mm
- net N$219: track 7.46 -> 24.0 mm
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
Commit message: functional state
Parts:
- moved C1 33.2 mm to (146.2, 39.6), turned to 90 degrees
- moved C2 31.2 mm to (153.4, 35.1)
- moved C103 31.2 mm to (152.8, 32.5)
- moved C102 28.8 mm to (143.7, 39.0), turned to 90 degrees
- moved U15 21.9 mm to (140.4, 28.6), turned to 315 degrees
- moved C109 19.0 mm to (143.7, 18.2), flipped to the bottom
- moved C113 18.7 mm to (144.3, 23.4), flipped to the bottom
- moved C111 16.9 mm to (126.1, 31.9)
- moved C107 16.9 mm to (126.1, 36.4)
- moved C6 16.7 mm to (146.2, 17.6), flipped to the bottom, turned to 270 degrees
- moved C7 16.3 mm to (122.8, 31.2)
- moved C117 16.3 mm to (126.1, 26.0), turned to 270 degrees
- moved C5 16.3 mm to (122.8, 37.0)
- moved C8 15.4 mm to (146.9, 24.1), flipped to the bottom, turned to 270 degrees
- moved C4 13.7 mm to (122.8, 25.4), turned to 270 degrees
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Routing:
- net SS_DAC_1: track 145.1 -> 180.9 mm
- net DVCC: track 1526.3 -> 1560.7 mm
- net DAC1_5: track 52.5 -> 22.4 mm
- net DAC1_6: track 55.2 -> 26.3 mm
- net DAC1_7: track 57.5 -> 29.7 mm
- net DAC1_4: track 46.2 -> 18.9 mm
- net DAC1_3: track 44.1 -> 17.3 mm
- net DAC1_2: track 42.3 -> 16.2 mm
- net DAC1_1: track 40.4 -> 16.5 mm
- net DAC1_0: track 38.6 -> 16.8 mm
- net N$151: track 7.46 -> 24.2 mm
- net N$152: track 63.3 -> 50.5 mm
- net VREF_1: track 29.4 -> 41.7 mm
- net DAC1_15: track 25.0 -> 13.9 mm
- net DAC1_14: track 23.6 -> 13.8 mm
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