File: electronics/Mainboard.brd (EAGLE design)
At the start: 310 x 150 mm, 225 parts, among them J1 JST_PH_B3B-PH-K-S(LF)(SN), J10 JST_PH_B3B-PH-K-S(LF)(SN), J11 JST_PH_B3B-PH-K-S(LF)(SN), J12 JST_PH_B3B-PH-K-S(LF)(SN), J13 JST_PH_B3B-PH-K-S(LF)(SN), J14 JST_PH_B3B-PH-K-S(LF)(SN), J15 JST_PH_B3B-PH-K-S(LF)(SN), J16 JST_PH_B3B-PH-K-S(LF)(SN), J17 JST_PH_B3B-PH-K-S(LF)(SN), J18 JST_PH_B3B-PH-K-S(LF)(SN), J19 JST_PH_B3B-PH-K-S(LF)(SN), J2 JST_PH_B3B-PH-K-S(LF)(SN), J20 JST_PH_B3B-PH-K-S(LF)(SN), J21 JST_PH_B3B-PH-K-S(LF)(SN), J22 JST_PH_B3B-PH-K-S(LF)(SN), J23 JST_PH_B3B-PH-K-S(LF)(SN), J24 JST_PH_B3B-PH-K-S(LF)(SN), J25 JST_PH_B3B-PH-K-S(LF)(SN), J26 JST_PH_B3B-PH-K-S(LF)(SN), J27 JST_PH_B3B-PH-K-S(LF)(SN), J28 JST_PH_B3B-PH-K-S(LF)(SN), J29 JST_PH_B3B-PH-K-S(LF)(SN), J3 JST_PH_B3B-PH-K-S(LF)(SN), J30 JST_PH_B3B-PH-K-S(LF)(SN), J31 JST_PH_B3B-PH-K-S(LF)(SN), J32 JST_PH_B3B-PH-K-S(LF)(SN), J4 JST_PH_B3B-PH-K-S(LF)(SN), J5 JST_PH_B3B-PH-K-S(LF)(SN), J6 JST_PH_B3B-PH-K-S(LF)(SN), J7 JST_PH_B3B-PH-K-S(LF)(SN), J8 JST_PH_B3B-PH-K-S(LF)(SN), J9 JST_PH_B3B-PH-K-S(LF)(SN), U15 AD5360BSTZ, U16 ADR425ARZ, U18 AD7730BRUZ, U19 AD5360BSTZ, U20 ADR425ARZ, U21 AD7730BRUZ, U22 STM32F103RCT6, U23 AD7730BRUZ, U24 AD7730BRUZ, U25 AD7730BRUZ, U26 AD7730BRUZ, U27 AD7730BRUZ, U28 AD7730BRUZ, U38 AD7730BRUZ, U39 AD7730BRUZ, U4 ADR421ARZ, U40 STM32F103RCT6, U41 AD7730BRUZ, U42 AD7730BRUZ, U43 AD7730BRUZ, U44 AD7730BRUZ, U45 AD7730BRUZ, U46 AD7730BRUZ, U5 AD7616BSTZ, U6 74AHC1G04GW/T1, U7 ADR421ARZ, U8 AD7616BSTZ, U9 74AHC1G04GW/T1, X1 22-23-2031, Y3 KC2520B-C1, Y4 ABM3B, Y7 KC2520B-C1, Y8 ABM3B

Commit message: switched to smd leds
Parts:
- LED1, LED2, LED3, LED4, LED5: device led:LED3MM -> led:CHIP-LED0603
- moved LED5 296.1 mm to (291.9, 120.2), turned to 0 degrees
- moved LED1 278.4 mm to (-3.90, 133.2), turned to 180 degrees
- moved LED3 5.99 mm to (280.1, 120.2), turned to 0 degrees
- moved LED4 5.99 mm to (286.0, 120.2), turned to 0 degrees
- moved LED2 5.99 mm to (274.3, 120.2), turned to 0 degrees
Connections:
- net +5V_CURR_LIM: now also LED2.A; no longer LED1.A
- net DVCC_CURR_LIM: now also LED3.A; no longer LED2.A
- net GND: now also LED1.C, LED2.C, LED3.C, LED4.C, LED5.C; no longer LED1.K, LED2.K, LED3.K, LED4.K, LED5.K
- net HB_CURR_LIM: now also LED1.A; no longer LED5.A
- net PG_CURR_LIM: now also LED4.A; no longer LED3.A
- net VDD_CURR_LIM: now also LED5.A; no longer LED4.A
Routing:
- net HB_CURR_LIM: track 4.70 -> 6.27 mm
- net VDD_CURR_LIM: track 22.5 -> 21.7 mm
- net PG_CURR_LIM: track 22.5 -> 21.7 mm
- net DVCC_CURR_LIM: track 22.5 -> 21.7 mm
- net +5V_CURR_LIM: track 22.5 -> 21.7 mm
Other:
- board text added: "Hitzmann 2018 rev. 2.1"
- board text removed: "Hitzmann 2018 rev. 2.0"
Changed lines of the file:
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@@
 <hole x="89.05" y="45.8" drill="5"/>
 <text x="17.55" y="20.15" size="1.778" layer="26" rot="MR0">Robot Controller Board</text>
-<text x="17.55" y="16.25" size="1.778" layer="26" rot="MR0">Hitzmann 2018 rev. 2.0</text>
+<text x="17.55" y="16.25" size="1.778" layer="26" rot="MR0">Hitzmann 2018 rev. 2.1</text>
 </plain>
 <attributes>
@@
 <attribute name="VALUE" x="279.655" y="135.872" size="1.27" layer="51" align="center"/>
 </element>
-<element name="LED3" library="led" library_urn="urn:adsk.eagle:library:259" package="LED3MM" package3d_urn="urn:adsk.eagle:package:15797/1" value="" x="286" y="121.55" smashed="yes" rot="R90">
-<attribute name="MF" value="VISHAY SEMICONDUCTOR" x="286" y="121.55" size="1.778" layer="27" rot="R90" display="off"/>
-<attribute name="NAME" x="283.669" y="119.555" size="1.27" layer="25" ratio="10" rot="R90"/>
-<attribute name="OC_FARNELL" value="1612435" x="286" y="121.55" size="1.778" layer="27" rot="R90" display="off"/>
-<attribute name="VALUE" x="287.651" y="123.455" size="1.27" layer="27" ratio="10" rot="R90"/>
-</element>
-<element name="LED2" library="led" library_urn="urn:adsk.eagle:library:259" package="LED3MM" package3d_urn="urn:adsk.eagle:package:15797/1" value="" x="280.15" y="121.55" smashed="yes" rot="R90">
-<attribute name="MF" value="VISHAY SEMICONDUCTOR" x="280.15" y="121.55" size="1.778" layer="27" rot="R90" display="off"/>
-<attribute name="NAME" x="277.819" y="119.555" size="1.27" layer="25" ratio="10" rot="R90"/>
-<attribute name="OC_FARNELL" value="1612435" x="280.15" y="121.55" size="1.778" layer="27" rot="R90" display="off"/>
-<attribute name="VALUE" x="281.801" y="123.455" size="1.27" layer="27" ratio="10" rot="R90"/>
-</element>
-<element name="LED1" library="led" library_urn="urn:adsk.eagle:library:259" package="LED3MM" package3d_urn="urn:adsk.eagle:package:15797/1" value="" x="274.3" y="121.55" smashed="yes" rot="R90">
-<attribute name="MF" value="VISHAY SEMICONDUCTOR" x="274.3" y="121.55" size="1.778" layer="27" rot="R90" display="off"/>
-<attribute name="NAME" x="271.969" y="119.555" size="1.27" layer="25" ratio="10" rot="R90"/>
-<attribute name="OC_FARNELL" value="1612435" x="274.3" y="121.55" size="1.778" layer="27" rot="R90" display="off"/>
-<attribute name="VALUE" x="275.951" y="123.455" size="1.27" layer="27" ratio="10" rot="R90"/>
-</element>
-<element name="LED4" library="led" library_urn="urn:adsk.eagle:library:259" package="LED3MM" package3d_urn="urn:adsk.eagle:package:15797/1" value="" x="291.85" y="121.55" smashed="yes" rot="R90">
-<attribute name="MF" value="VISHAY SEMICONDUCTOR" x="291.85" y="121.55" size="1.778" layer="27" rot="R90" display="off"/>
-<attribute name="NAME" x="289.519" y="119.555" size="1.27" layer="25" ratio="10" rot="R90"/>
-<attribute name="OC_FARNELL" value="1612435" x="291.85" y="121.55" size="1.778" layer="27" rot="R90" display="off"/>
-<attribute name="VALUE" x="293.501" y="123.455" size="1.27" layer="27" ratio="10" rot="R90"/>
-</element>
 <element name="R1" library="resistor" library_urn="urn:adsk.eagle:library:348" package="R0805" package3d_urn="urn:adsk.eagle:package:26059/1" value="220" x="286" y="96.85" smashed="yes" rot="R270">
 <attribute name="NAME" x="287.27" y="97.485" size="1.27" layer="25" rot="R270"/>
@@
 <attribute name="VALUE" x="-7.68" y="54.51" size="1.27" layer="27" ratio="10" rot="R270"/>
 </element>
-<element name="LED5" library="led" library_urn="urn:adsk.eagle:library:259" package="LED3MM" package3d_urn="urn:adsk.eagle:package:15797/1" value="" x="-3.9" y="133.9" smashed="yes" rot="R270">
-<attribute name="MF" value="VISHAY SEMICONDUCTOR" x="-3.9" y="133.9" size="1.778" layer="27" rot="R270" display="off"/>
-<attribute name="NAME" x="-6.881" y="132.555" size="1.27" layer="25" ratio="10" rot="R90"/>
-<attribute name="OC_FARNELL" value="1612435" x="-3.9" y="133.9" size="1.778" layer="27" rot="R270" display="off"/>
-<attribute name="VALUE" x="-5.551" y="131.995" size="1.27" layer="27" ratio="10" rot="R270"/>
-</element>
 <element name="R11" library="resistor" library_urn="urn:adsk.eagle:library:348" package="R0805" package3d_urn="urn:adsk.eagle:package:26059/1" value="330" x="1.2" y="136.5" smashed="yes">
 <attribute name="NAME" x="-0.735" y="137.77" size="1.27" layer="25"/>
@@
 <attribute name="VALUE" x="21.15" y="27.35" size="1.27" layer="27" rot="R90"/>
 </element>
+<element name="LED1" library="led" library_urn="urn:adsk.eagle:library:259" package="CHIP-LED0603" package3d_urn="urn:adsk.eagle:package:15819/3" value="" x="-3.9" y="133.25" smashed="yes" rot="R180">
+<attribute name="NAME" x="-6.515" y="136.485" size="1.27" layer="25" rot="R270"/>
+<attribute name="VALUE" x="-5.805" y="133.885" size="1.27" layer="27" rot="R270"/>
+</element>
+<element name="LED5" library="led" library_urn="urn:adsk.eagle:library:259" package="CHIP-LED0603" package3d_urn="urn:adsk.eagle:package:15819/3" value="" x="291.85" y="120.25"/>
+<element name="LED2" library="led" library_urn="urn:adsk.eagle:library:259" package="CHIP-LED0603" package3d_urn="urn:adsk.eagle:package:15819/3" value="" x="274.3" y="120.25"/>
+<element name="LED3" library="led" library_urn="urn:adsk.eagle:library:259" package="CHIP-LED0603" package3d_urn="urn:adsk.eagle:package:15819/3" value="" x="280.15" y="120.25"/>
+<element name="LED4" library="led" library_urn="urn:adsk.eagle:library:259" package="CHIP-LED0603" package3d_urn="urn:adsk.eagle:package:15819/3" value="" x="286" y="120.25"/>
 </elements>
 <signals>
@@
 <contactref element="U8" pad="10"/>
 <contactref element="S1" pad="3"/>
-<contactref element="LED3" pad="K"/>
-<contactref element="LED2" pad="K"/>
-<contactref element="LED1" pad="K"/>
-<contactref element="LED4" pad="K"/>
 <contactref element="X1" pad="3"/>
-<contactref element="LED5" pad="K"/>
 <contactref element="C1" pad="-"/>
 <contactref element="C2" pad="-"/>
@@
 <via x="113.75" y="104.65" extent="1-16" drill="0.3048"/>
 <via x="113.75" y="102.7" extent="1-16" drill="0.3048"/>
+<contactref element="LED1" pad="C"/>
+<contactref element="LED5" pad="C"/>
+<contactref element="LED2" pad="C"/>
+<contactref element="LED3" pad="C"/>
+<contactref element="LED4" pad="C"/>
 </signal>
 <signal name="MISO">
@@
 </signal>
 <signal name="PG_CURR_LIM">
-<contactref element="LED3" pad="A"/>
 <contactref element="R1" pad="1"/>
-<wire x1="286" y1="120.28" x2="286" y2="97.8" width="0.4064" layer="1"/>
+<contactref element="LED4" pad="A"/>
+<wire x1="286" y1="97.8" x2="286" y2="119.5" width="0.4064" layer="1"/>
 </signal>
 <signal name="DVCC_CURR_LIM">
-<contactref element="LED2" pad="A"/>
 <contactref element="R3" pad="1"/>
-<wire x1="280.15" y1="120.28" x2="280.15" y2="97.8" width="0.4064" layer="1"/>
+<contactref element="LED3" pad="A"/>
+<wire x1="280.15" y1="97.8" x2="280.15" y2="119.5" width="0.4064" layer="1"/>
 </signal>
 <signal name="+5V_CURR_LIM">
-<contactref element="LED1" pad="A"/>
 <contactref element="R5" pad="1"/>
-<wire x1="274.3" y1="120.28" x2="274.3" y2="97.8" width="0.4064" layer="1"/>
+<contactref element="LED2" pad="A"/>
+<wire x1="274.3" y1="97.8" x2="274.3" y2="119.5" width="0.4064" layer="1"/>
 </signal>
 <signal name="VDD_CURR_LIM">
-<contactref element="LED4" pad="A"/>
 <contactref element="R10" pad="1"/>
-<wire x1="291.85" y1="120.28" x2="291.85" y2="97.8" width="0.4064" layer="1"/>
+<contactref element="LED5" pad="A"/>
+<wire x1="291.85" y1="97.8" x2="291.85" y2="119.5" width="0.4064" layer="1"/>
 </signal>
 <signal name="RPI_PWR">
@@
 </signal>
 <signal name="HB_CURR_LIM">
-<contactref element="LED5" pad="A"/>
 <contactref element="R11" pad="1"/>
-<wire x1="0.25" y1="136.5" x2="-2.57" y2="136.5" width="0.4064" layer="1"/>
-<wire x1="-2.57" y1="136.5" x2="-3.9" y2="135.17" width="0.4064" layer="1"/>
+<contactref element="LED1" pad="A"/>
+<wire x1="-3.25" y1="136.5" x2="-3.9" y2="135.85" width="0.4064" layer="1"/>
+<wire x1="-3.9" y1="135.85" x2="-3.9" y2="134" width="0.4064" layer="1"/>
+<wire x1="0.25" y1="136.5" x2="-3.25" y2="136.5" width="0.4064" layer="1"/>
 </signal>
 <signal name="HEARTBEAT">

Commit message: re-routed spi bus
Parts:
- moved S8 8.47 mm to (160.6, 119.0)
- moved JP1 3.90 mm to (12.2, 150.9)
- moved SV1 2.60 mm to (35.1, 144.3)
- moved C13 1.95 mm to (231.9, 117.5)
- moved C54 1.95 mm to (231.9, 40.8)
- moved S6 1.30 mm to (157.3, 48.1)
- moved U6 0.65 mm to (31.2, 119.0)
- moved U9 0.65 mm to (31.2, 41.0)
- moved C3 0.65 mm to (98.2, 18.4)
- moved C16 0.65 mm to (221.2, 133.7)
Connections:
- net CONVST: now also SV1.11; no longer SV1.16
- net LDAC: now also SV1.35; no longer SV1.18
- net SS_ADC_2: now also SV1.13; no longer SV1.31
- net SS_DAC_1: now also SV1.36; no longer SV1.35
- net SS_DAC_2: now also SV1.40; no longer SV1.36
- net SS_LC_1: now also SV1.38; no longer SV1.32
- net SS_LC_2: now also SV1.37; no longer SV1.26
Routing:
- net MOSI: track 680.5 -> 625.6 mm, vias 9 -> 11
- net MISO: track 675.8 -> 636.1 mm, vias 9 -> 11
- net DVCC: track 1566.5 -> 1542.2 mm
- net SS_LC_2: track 200.7 -> 183.2 mm, vias 3 -> 1
- net PSU_ENABLE: track 117.5 -> 100.3 mm
- net SS_DAC_2: track 121.0 -> 134.2 mm
- net SS_DAC_1: track 179.9 -> 191.8 mm, vias 2 -> 3
- net LDAC: track 238.7 -> 232.4 mm, vias 3 -> 6
- net CONVST: track 160.4 -> 154.4 mm, vias 1 -> 2
- net SS_LC_1: track 244.5 -> 248.8 mm
- net VDD: track 1027.6 -> 1028.8 mm, vias 20 -> 19
- net DAC_1_RST: track 47.2 -> 48.3 mm
- net DAC_2_RST: track 47.6 -> 48.6 mm
- net SCLK: track 656.7 -> 657.7 mm, vias 6 -> 11
- net VSS: track 484.6 -> 485.5 mm
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Other:
- board size 310 x 150 mm -> 310 x 155 mm

Commit message: reworked vias
Parts:
- added Q1: (no value), transistor-npn:SOT23-BEC
- R1: value 220 -> 68
- moved R5 13.7 mm to (274.3, 110.5)
- moved S2 9.66 mm to (72.8, 119.0)
- moved R1 7.15 mm to (286.0, 104.0)
- moved R10 7.15 mm to (291.9, 104.0)
- moved R3 7.15 mm to (280.1, 104.0)
- moved S3 6.50 mm to (72.8, 48.1)
- moved S6 3.25 mm to (160.6, 48.1)
- moved C28 0.65 mm to (19.8, 107.0)
- moved C30 0.65 mm to (19.8, 28.9)
- moved C36 0.65 mm to (22.1, 106.3)
- moved C67 0.65 mm to (22.1, 28.3)
Connections:
- new net POWER_GOOD_SUPP: Q1.E, R1.2
- net DVCC: now also Q1.C
- net POWER_GOOD: now also Q1.B; no longer R1.2
Routing:
- net +5V: track 1379.6 -> 1393.3 mm
- net +5V_CURR_LIM: track 21.7 -> 8.05 mm
- net DVCC: track 1542.2 -> 1554.7 mm
- net VDD: track 1028.8 -> 1036.0 mm
- net VDD_CURR_LIM: track 21.7 -> 14.5 mm
- net PG_CURR_LIM: track 21.7 -> 14.5 mm
- net DVCC_CURR_LIM: track 21.7 -> 14.5 mm
- net POWER_GOOD_SUPP: track 0.00 -> 5.95 mm
- net ADC_1_RST: track 24.6 -> 28.6 mm
- net DAC_1_RST: track 48.3 -> 51.6 mm
- net ADC_2_RST: track 24.6 -> 25.6 mm
- net DAC_2_CLR: track 22.0 -> 22.9 mm
- net POWER_GOOD: track 39.5 -> 38.8 mm
- net DAC_1_CLR: track 22.6 -> 23.2 mm

Commit message: added more gnd connecting vias
Parts:
- added R12: 1k, resistor:R0805
- moved R1 6.50 mm to (286.0, 110.5)
- moved Q1 3.90 mm to (284.9, 100.0)
- moved R10 2.60 mm to (291.9, 106.6)
- moved R3 2.60 mm to (280.1, 106.6)
- moved C53 2.17 mm to (220.2, 39.1), turned to 0 degrees
- moved C15 2.17 mm to (220.2, 115.8), turned to 180 degrees
- moved C12 1.45 mm to (214.0, 122.9)
- moved C57 1.45 mm to (214.0, 46.2)
- moved C76 0.11 mm to (57.9, 34.6)
- moved C45 0.10 mm to (58.0, 112.7)
Connections:
- new net PG_SIG: Q1.B, R12.1
- net POWER_GOOD: now also R12.2; no longer Q1.B
Routing:
- net DVCC: track 1554.7 -> 1561.3 mm
- net PG_CURR_LIM: track 14.5 -> 8.05 mm
- net PG_SIG: track 0.00 -> 3.90 mm
- net VDD_CURR_LIM: track 14.5 -> 12.0 mm
- net POWER_GOOD_SUPP: track 5.95 -> 8.55 mm
- net DVCC_CURR_LIM: track 14.5 -> 12.0 mm
- net VDD: track 1036.0 -> 1038.6 mm
- net POWER_GOOD: track 38.8 -> 36.9 mm

Commit message: cleaned pcb and updated firmware version
Routing:
- net +5V: track 1393.3 -> 1390.4 mm
- net DVCC: track 1561.3 -> 1559.1 mm
- net LC_1_SPI1_MOSI: track 113.5 -> 113.0 mm
