File: electronics/Mainboard.sch (EAGLE design)
At the start: 226 parts, among them J1 JST_PH_B3B-PH-K-S(LF)(SN), J10 JST_PH_B3B-PH-K-S(LF)(SN), J11 JST_PH_B3B-PH-K-S(LF)(SN), J12 JST_PH_B3B-PH-K-S(LF)(SN), J13 JST_PH_B3B-PH-K-S(LF)(SN), J14 JST_PH_B3B-PH-K-S(LF)(SN), J15 JST_PH_B3B-PH-K-S(LF)(SN), J16 JST_PH_B3B-PH-K-S(LF)(SN), J17 JST_PH_B3B-PH-K-S(LF)(SN), J18 JST_PH_B3B-PH-K-S(LF)(SN), J19 JST_PH_B3B-PH-K-S(LF)(SN), J2 JST_PH_B3B-PH-K-S(LF)(SN), J20 JST_PH_B3B-PH-K-S(LF)(SN), J21 JST_PH_B3B-PH-K-S(LF)(SN), J22 JST_PH_B3B-PH-K-S(LF)(SN), J23 JST_PH_B3B-PH-K-S(LF)(SN), J24 JST_PH_B3B-PH-K-S(LF)(SN), J25 JST_PH_B3B-PH-K-S(LF)(SN), J26 JST_PH_B3B-PH-K-S(LF)(SN), J27 JST_PH_B3B-PH-K-S(LF)(SN), J28 JST_PH_B3B-PH-K-S(LF)(SN), J29 JST_PH_B3B-PH-K-S(LF)(SN), J3 JST_PH_B3B-PH-K-S(LF)(SN), J30 JST_PH_B3B-PH-K-S(LF)(SN), J31 JST_PH_B3B-PH-K-S(LF)(SN), J32 JST_PH_B3B-PH-K-S(LF)(SN), J33 B4B-PH-K-S(LF)(SN), J34 B4B-PH-K-S(LF)(SN), J35 B4B-PH-K-S(LF)(SN), J36 B4B-PH-K-S(LF)(SN), J37 B4B-PH-K-S(LF)(SN), J38 B4B-PH-K-S(LF)(SN), J39 B4B-PH-K-S(LF)(SN), J4 JST_PH_B3B-PH-K-S(LF)(SN), J40 B4B-PH-K-S(LF)(SN), J41 B4B-PH-K-S(LF)(SN), J42 B4B-PH-K-S(LF)(SN), J43 B4B-PH-K-S(LF)(SN), J44 B4B-PH-K-S(LF)(SN), J45 B4B-PH-K-S(LF)(SN), J46 B4B-PH-K-S(LF)(SN), J47 B4B-PH-K-S(LF)(SN), J48 B4B-PH-K-S(LF)(SN), J49 B4B-PH-K-S(LF)(SN), J5 JST_PH_B3B-PH-K-S(LF)(SN), J50 B4B-PH-K-S(LF)(SN), J51 B4B-PH-K-S(LF)(SN), J52 B4B-PH-K-S(LF)(SN), J53 B4B-PH-K-S(LF)(SN), J54 B4B-PH-K-S(LF)(SN), J55 B4B-PH-K-S(LF)(SN), J56 B4B-PH-K-S(LF)(SN), J57 B4B-PH-K-S(LF)(SN), J58 B4B-PH-K-S(LF)(SN), J59 B4B-PH-K-S(LF)(SN), J6 JST_PH_B3B-PH-K-S(LF)(SN), J60 B4B-PH-K-S(LF)(SN), J61 B4B-PH-K-S(LF)(SN), J62 B4B-PH-K-S(LF)(SN), J63 B4B-PH-K-S(LF)(SN), J64 B4B-PH-K-S(LF)(SN), J7 JST_PH_B3B-PH-K-S(LF)(SN), J8 JST_PH_B3B-PH-K-S(LF)(SN), J9 JST_PH_B3B-PH-K-S(LF)(SN), Q1 BCF29SMD, U1 AMP-5103309-7-34PIN_5103309-7, U15 AD5360BSTZ, U16 ADR425ARZ, U18 AD7730BRUZ, U19 AD5360BSTZ, U2 AMP-5103309-7-34PIN_5103309-7, U20 ADR425ARZ, U21 AD7730BRUZ, U22 STM32F103RCT6, U23 AD7730BRUZ, U24 AD7730BRUZ, U25 AD7730BRUZ, U26 AD7730BRUZ, U27 AD7730BRUZ, U28 AD7730BRUZ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

Commit message: added more gnd connecting vias
Parts:
- added R12: 1k, resistor:R-EU_R0805
Connections:
- new net PG_SIG: Q1.B, R12.1
- net POWER_GOOD: now also R12.2; no longer Q1.B
Changed lines of the file:
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@@
 <part name="LED4" library="led" library_urn="urn:adsk.eagle:library:259" deviceset="LED" device="CHIP-LED0603" package3d_urn="urn:adsk.eagle:package:15819/3"/>
 <part name="Q1" library="transistor-npn" library_urn="urn:adsk.eagle:library:398" deviceset="BCF29*" device="SMD" package3d_urn="urn:adsk.eagle:package:28990/2" value=""/>
+<part name="R12" library="resistor" library_urn="urn:adsk.eagle:library:348" deviceset="R-EU_" device="R0805" package3d_urn="urn:adsk.eagle:package:26059/1" value="1k"/>
 </parts>
 <sheets>
@@
 <attribute name="VALUE" x="292.1" y="279.4" size="1.778" layer="96"/>
 </instance>
+<instance part="R12" gate="G$1" x="289.56" y="274.32" smashed="yes" rot="R180">
+<attribute name="NAME" x="290.83" y="272.8214" size="1.778" layer="95" rot="R180"/>
+<attribute name="VALUE" x="290.83" y="277.622" size="1.778" layer="96" rot="R180"/>
+</instance>
 </instances>
 <busses>
@@
 <wire x1="403.86" y1="256.54" x2="396.24" y2="256.54" width="0.1524" layer="91"/>
 <label x="386.08" y="256.54" size="1.778" layer="95"/>
+<wire x1="396.24" y1="256.54" x2="386.08" y2="256.54" width="0.1524" layer="91"/>
 </segment>
 </net>
@@
 </segment>
 <segment>
-<pinref part="Q1" gate="G$1" pin="B"/>
-<wire x1="299.72" y1="274.32" x2="276.86" y2="274.32" width="0.1524" layer="91"/>
-<label x="276.86" y="274.32" size="1.778" layer="95"/>
+<label x="266.7" y="274.32" size="1.778" layer="95"/>
+<pinref part="R12" gate="G$1" pin="2"/>
+<wire x1="269.24" y1="274.32" x2="284.48" y2="274.32" width="0.1524" layer="91"/>
 </segment>
 </net>
@@
 </segment>
 </net>
+<net name="PG_SIG" class="0">
+<segment>
+<pinref part="R12" gate="G$1" pin="1"/>
+<pinref part="Q1" gate="G$1" pin="B"/>
+<wire x1="294.64" y1="274.32" x2="299.72" y2="274.32" width="0.1524" layer="91"/>
+<label x="299.72" y="274.32" size="1.778" layer="95" rot="R90"/>
+</segment>
+</net>
